File: crush-pcb.kicad_sch (KiCad schematic)
At the start: 2 parts, among them U1 Teensy4.1

Commit message: 2/26 Work as a team
Parts:
- added J1: TSW-108-07-G-T, SAMTEC_TSW-108-07-G-T, symbol 3x8 Header:TSW-108-07-G-T
Other:
- sheet I2C Level Shifter ports: added 3V3, 5V; removed none
- note added: "PWM2-PWM9 = thrusters"
Changed lines of the file:
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@@
+    (stroke (width 0) (type default))
+  )
+  (wire (pts (xy 151.13 11.43) (xy 154.94 11.43))
+    (stroke (width 0) (type default))
+  )
+  (wire (pts (xy 182.88 15.24) (xy 179.07 15.24))
     (stroke (width 0) (type default))
   )
@@
     (stroke (width 0) (type default))
   )
+  (wire (pts (xy 151.13 15.24) (xy 154.94 15.24))
+    (stroke (width 0) (type default))
+  )
+  (wire (pts (xy 182.88 11.43) (xy 179.07 11.43))
+    (stroke (width 0) (type default))
+  )
   (wire (pts (xy 10.16 97.79) (xy 10.16 20.32))
     (stroke (width 0) (type default))
@@
     (stroke (width 0) (type default))
   )
+  (text "PWM2-PWM9 = thrusters\n" (at 13.97 48.26 90)
+    (effects (font (size 1.27 1.27)) (justify left bottom))
+  )
   (global_label "PWM2" (shape input) (at 25.4 27.94 180) (fields_autoplaced)
     (effects (font (size 1.27 1.27)) (justify right))
@@
     )
   )
+  (global_label "SDA_3V3" (shape input) (at 151.13 15.24 180) (fields_autoplaced)
+    (effects (font (size 1.27 1.27)) (justify right))
+    (property "Intersheetrefs" "${INTERSHEET_REFS}" (at 140.1809 15.24 0)
+      (effects (font (size 1.27 1.27)) (justify right) hide)
+    )
+  )
   (global_label "UART_RX" (shape input) (at 25.4 22.86 180) (fields_autoplaced)
     (effects (font (size 1.27 1.27)) (justify right))
@@
     )
   )
+  (global_label "SCL_3V3" (shape input) (at 151.13 11.43 180) (fields_autoplaced)
+    (effects (font (size 1.27 1.27)) (justify right))
+    (property "Intersheetrefs" "${INTERSHEET_REFS}" (at 140.2414 11.43 0)
+      (effects (font (size 1.27 1.27)) (justify right) hide)
+    )
+  )
   (global_label "SPI_SCK" (shape input) (at 81.28 53.34 0) (fields_autoplaced)
     (effects (font (size 1.27 1.27)) (justify left))
@@
     )
   )
+  (global_label "SCL_5V" (shape input) (at 182.88 11.43 0) (fields_autoplaced)
+    (effects (font (size 1.27 1.27)) (justify left))
+    (property "Intersheetrefs" "${INTERSHEET_REFS}" (at 192.5591 11.43 0)
+      (effects (font (size 1.27 1.27)) (justify left) hide)
+    )
+  )
   (global_label "USB_5V" (shape input) (at 120.65 10.16 0) (fields_autoplaced)
     (effects (font (size 1.27 1.27)) (justify left))
@@
     (effects (font (size 1.27 1.27)) (justify left))
     (property "Intersheetrefs" "${INTERSHEET_REFS}" (at 91.7364 40.5606 0)
+      (effects (font (size 1.27 1.27)) (justify left) hide)
+    )
+  )
+  (global_label "SDA_5V" (shape input) (at 182.88 15.24 0) (fields_autoplaced)
+    (effects (font (size 1.27 1.27)) (justify left))
+    (property "Intersheetrefs" "${INTERSHEET_REFS}" (at 192.6196 15.24 0)
       (effects (font (size 1.27 1.27)) (justify left) hide)
     )
@@
         (path "/74b566fe-9d71-4817-95ed-d472d647f8c8"
           (reference "J?") (unit 1)
-        )
-      )
-    )
-  )
-  (symbol (lib_id "crush-pcb-altium-import:GND") (at 10.16 105.41 0) (unit 1)
-    (in_bom yes) (on_board yes) (dnp no)
-    (property "Reference" "#PWR?" (at 10.16 100.33 0)
-      (effects (font (size 1.27 1.27)) hide)
-    )
-    (property "Value" "GND" (at 6.35 105.41 0)
-      (effects (font (size 1.27 1.27)) hide)
-    )
-    (property "Footprint" "" (at 10.16 105.41 0)
-      (effects (font (size 1.27 1.27)) hide)
-    )
-    (property "Datasheet" "" (at 10.16 105.41 0)
-      (effects (font (size 1.27 1.27)) hide)
-    )
-    (pin "")
-    (instances
-      (project "crush-pcb"
-        (path "/74b566fe-9d71-4817-95ed-d472d647f8c8"
-          (reference "#PWR?") (unit 1)
         )
       )
@@
     )
   )
-  (symbol (lib_id "crush-pcb-altium-import:GND") (at 113.03 25.4 0) (unit 1)
-    (in_bom yes) (on_board yes) (dnp no)
-    (property "Reference" "#PWR?" (at 113.03 20.32 0)
-      (effects (font (size 1.27 1.27)) hide)
-    )
-    (property "Value" "GND" (at 109.22 25.4 0)
-      (effects (font (size 1.27 1.27)) hide)
+  (symbol (lib_id "3x8 Header:TSW-108-07-G-T") (at 167.64 55.88 0) (unit 1)
+    (in_bom yes) (on_board yes) (dnp no) (fields_autoplaced)
+    (property "Reference" "J1" (at 167.64 29.21 0)
+      (effects (font (size 1.27 1.27)))
+    )
+    (property "Value" "TSW-108-07-G-T" (at 167.64 31.75 0)
+      (effects (font (size 1.27 1.27)))
+    )
+    (property "Footprint" "SAMTEC_TSW-108-07-G-T" (at 167.64 55.88 0)
+      (effects (font (size 1.27 1.27)) (justify bottom) hide)
+    )
+    (property "Datasheet" "" (at 167.64 55.88 0)
+      (effects (font (size 1.27 1.27)) hide)
+    )
+    (property "STANDARD" "Manufacturer Recommendations" (at 167.64 55.88 0)
+      (effects (font (size 1.27 1.27)) (justify bottom) hide)
+    )
+    (property "PARTREV" "R" (at 167.64 55.88 0)
+      (effects (font (size 1.27 1.27)) (justify bottom) hide)
+    )
+    (property "MANUFACTURER" "Samtec" (at 167.64 55.88 0)
+      (effects (font (size 1.27 1.27)) (justify bottom) hide)
+    )
+    (pin "01")
+    (pin "02")
+    (pin "03")
+    (pin "04")
+    (pin "05")
+    (pin "06")
+    (pin "07")
+    (pin "08")
+    (pin "09")
+    (pin "10")
+    (pin "11")
+    (pin "12")
+    (pin "13")
+    (pin "14")
+    (pin "15")
+    (pin "16")
+    (pin "17")
+    (pin "18")
+    (pin "19")
+    (pin "20")
+    (pin "21")
+    (pin "22")
+    (pin "23")
+    (pin "24")
+    (instances
+      (project "crush-pcb"
+        (path "/74b566fe-9d71-4817-95ed-d472d647f8c8"
+          (reference "J1") (unit 1)
+        )
+      )
+    )
+  )
+  (symbol (lib_id "power:GND") (at 113.03 25.4 0) (unit 1)
+    (in_bom yes) (on_board yes) (dnp no) (fields_autoplaced)
+    (property "Reference" "#PWR03" (at 113.03 31.75 0)
+      (effects (font (size 1.27 1.27)) hide)
+    )
+    (property "Value" "GND" (at 113.03 30.48 0)
+      (effects (font (size 1.27 1.27)))
     )
     (property "Footprint" "" (at 113.03 25.4 0)
@@
       (effects (font (size 1.27 1.27)) hide)
     )
-    (pin "")
-    (instances
-      (project "crush-pcb"
-        (path "/74b566fe-9d71-4817-95ed-d472d647f8c8"
-          (reference "#PWR?") (unit 1)
+    (pin "1")
+    (instances
+      (project "crush-pcb"
+        (path "/74b566fe-9d71-4817-95ed-d472d647f8c8"
+          (reference "#PWR03") (unit 1)
         )
       )
@@
     )
   )
-  (symbol (lib_id "crush-pcb-altium-import:GND") (at 99.06 85.09 0) (unit 1)
-    (in_bom yes) (on_board yes) (dnp no)
-    (property "Reference" "#PWR?" (at 99.06 80.01 0)
-      (effects (font (size 1.27 1.27)) hide)
-    )
-    (property "Value" "GND" (at 95.25 85.09 0)
-      (effects (font (size 1.27 1.27)) hide)
+  (symbol (lib_id "power:GND") (at 10.16 105.41 0) (unit 1)
+    (in_bom yes) (on_board yes) (dnp no) (fields_autoplaced)
+    (property "Reference" "#PWR01" (at 10.16 111.76 0)
+      (effects (font (size 1.27 1.27)) hide)
+    )
+    (property "Value" "GND" (at 10.16 110.49 0)
+      (effects (font (size 1.27 1.27)))
+    )
+    (property "Footprint" "" (at 10.16 105.41 0)
+      (effects (font (size 1.27 1.27)) hide)
+    )
+    (property "Datasheet" "" (at 10.16 105.41 0)
+      (effects (font (size 1.27 1.27)) hide)
+    )
+    (pin "1")
+    (instances
+      (project "crush-pcb"
+        (path "/74b566fe-9d71-4817-95ed-d472d647f8c8"
+          (reference "#PWR01") (unit 1)
+        )
+      )
+    )
+  )
+  (symbol (lib_id "power:GND") (at 99.06 85.09 0) (unit 1)
+    (in_bom yes) (on_board yes) (dnp no) (fields_autoplaced)
+    (property "Reference" "#PWR02" (at 99.06 91.44 0)
+      (effects (font (size 1.27 1.27)) hide)
+    )
+    (property "Value" "GND" (at 99.06 90.17 0)
+      (effects (font (size 1.27 1.27)))
     )
     (property "Footprint" "" (at 99.06 85.09 0)
@@
       (effects (font (size 1.27 1.27)) hide)
     )
-    (pin "")
-    (instances
-      (project "crush-pcb"
-        (path "/74b566fe-9d71-4817-95ed-d472d647f8c8"
-          (reference "#PWR?") (unit 1)
-        )
-      )
-    )
-  )
-  (sheet (at 152.4 13.97) (size 24.13 11.43) (fields_autoplaced)
+    (pin "1")
+    (instances
+      (project "crush-pcb"
+        (path "/74b566fe-9d71-4817-95ed-d472d647f8c8"
+          (reference "#PWR02") (unit 1)
+        )
+      )
+    )
+  )
+  (sheet (at 154.94 5.08) (size 24.13 12.7) (fields_autoplaced)
     (stroke (width 0.1524) (type solid))
     (fill (color 0 0 0 0.0000))
-    (property "Sheetname" "I2C Level Shifter" (at 152.4 13.2584 0)
+    (property "Sheetname" "I2C Level Shifter" (at 154.94 4.3684 0)
       (effects (font (size 1.27 1.27)) (justify left bottom))
     )
-    (property "Sheetfile" "i2c_level_shifter.kicad_sch" (at 152.4 25.9846 0)
+    (property "Sheetfile" "i2c_level_shifter.kicad_sch" (at 154.94 18.3646 0)
       (effects (font (size 1.27 1.27)) (justify left top))
     )
-    (pin "SCL_3V3" bidirectional (at 152.4 19.05 180)
+    (pin "SCL_3V3" bidirectional (at 154.94 11.43 180)
       (effects (font (size 1.27 1.27)) (justify left))
     )
-    (pin "SDA_3V3" bidirectional (at 152.4 22.86 180)
+    (pin "SDA_3V3" bidirectional (at 154.94 15.24 180)
       (effects (font (size 1.27 1.27)) (justify left))
     )
-    (pin "SDA_5V" bidirectional (at 176.53 22.86 0)
+    (pin "SDA_5V" bidirectional (at 179.07 15.24 0)
       (effects (font (size 1.27 1.27)) (justify right))
     )
-    (pin "SCL_5V" bidirectional (at 176.53 19.05 0)
+    (pin "SCL_5V" bidirectional (at 179.07 11.43 0)
       (effects (font (size 1.27 1.27)) (justify right))
     )
+    (pin "3V3" input (at 154.94 7.62 180)
+      (effects (font (size 1.27 1.27)) (justify left))
+    )
+    (pin "5V" input (at 179.07 7.62 0)
+      (effects (font (size 1.27 1.27)) (justify right))
+    )
