File: crush-pcb.kicad_sch (KiCad schematic)
At the start: 3 parts, among them J1 3x8 Header, U1 Teensy4.1

Commit message: baby change to test committing
Connections:
- net GND: now also J1.01, J1.03, J1.04, J1.06, J1.07, J1.09, J1.10, J1.12, J1.13, J1.15, J1.16, J1.18, J1.19, J1.21, J1.22, J1.24
Changed lines of the file:
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@@
     (rev "1")
   )
+  (junction (at 111.76 48.26) (diameter 0) (color 0 0 0 0)
+  )
+  (junction (at 111.76 81.28) (diameter 0) (color 0 0 0 0)
+  )
+  (junction (at 111.76 73.66) (diameter 0) (color 0 0 0 0)
+  )
+  (junction (at 111.76 50.8) (diameter 0) (color 0 0 0 0)
+  )
+  (junction (at 111.76 76.2) (diameter 0) (color 0 0 0 0)
+  )
+  (junction (at 111.76 43.18) (diameter 0) (color 0 0 0 0)
+  )
   (junction (at 10.16 97.79) (diameter 0) (color 0 0 0 0)
   )
+  (junction (at 111.76 71.12) (diameter 0) (color 0 0 0 0)
+  )
+  (junction (at 111.76 63.5) (diameter 0) (color 0 0 0 0)
+  )
   (junction (at 99.06 55.88) (diameter 0) (color 0 0 0 0)
   )
+  (junction (at 111.76 66.04) (diameter 0) (color 0 0 0 0)
+  )
   (junction (at 10.16 100.33) (diameter 0) (color 0 0 0 0)
+  )
+  (junction (at 111.76 55.88) (diameter 0) (color 0 0 0 0)
+  )
+  (junction (at 111.76 78.74) (diameter 0) (color 0 0 0 0)
+  )
+  (junction (at 111.76 53.34) (diameter 0) (color 0 0 0 0)
+  )
+  (junction (at 111.76 68.58) (diameter 0) (color 0 0 0 0)
+  )
+  (junction (at 111.76 58.42) (diameter 0) (color 0 0 0 0)
+  )
+  (junction (at 111.76 45.72) (diameter 0) (color 0 0 0 0)
   )
   (no_connect (at 120.65 20.32))
@@
     (stroke (width 0) (type default))
   )
+  (wire (pts (xy 111.76 43.18) (xy 111.76 45.72))
+    (stroke (width 0) (type default))
+  )
+  (wire (pts (xy 111.76 63.5) (xy 111.76 66.04))
+    (stroke (width 0) (type default))
+  )
   (wire (pts (xy 10.16 97.79) (xy 25.4 97.79))
     (stroke (width 0) (type default))
   )
+  (wire (pts (xy 111.76 48.26) (xy 111.76 50.8))
+    (stroke (width 0) (type default))
+  )
   (wire (pts (xy 148.59 6.35) (xy 148.59 11.43))
     (stroke (width 0) (type default))
   )
+  (wire (pts (xy 111.76 71.12) (xy 111.76 73.66))
+    (stroke (width 0) (type default))
+  )
+  (wire (pts (xy 111.76 73.66) (xy 111.76 76.2))
+    (stroke (width 0) (type default))
+  )
+  (wire (pts (xy 111.76 53.34) (xy 111.76 55.88))
+    (stroke (width 0) (type default))
+  )
   (wire (pts (xy 99.06 22.86) (xy 99.06 55.88))
     (stroke (width 0) (type default))
   )
+  (wire (pts (xy 111.76 45.72) (xy 111.76 48.26))
+    (stroke (width 0) (type default))
+  )
+  (wire (pts (xy 111.76 40.64) (xy 111.76 43.18))
+    (stroke (width 0) (type default))
+  )
   (wire (pts (xy 88.9 13.97) (xy 88.9 20.32))
     (stroke (width 0) (type default))
@@
     (stroke (width 0) (type default))
   )
+  (wire (pts (xy 111.76 58.42) (xy 111.76 63.5))
+    (stroke (width 0) (type default))
+  )
   (wire (pts (xy 151.13 19.05) (xy 154.94 19.05))
     (stroke (width 0) (type default))
@@
     (stroke (width 0) (type default))
   )
+  (wire (pts (xy 111.76 76.2) (xy 111.76 78.74))
+    (stroke (width 0) (type default))
+  )
   (wire (pts (xy 182.88 15.24) (xy 179.07 15.24))
     (stroke (width 0) (type default))
   )
+  (wire (pts (xy 111.76 81.28) (xy 111.76 86.36))
+    (stroke (width 0) (type default))
+  )
   (wire (pts (xy 187.96 6.35) (xy 187.96 11.43))
     (stroke (width 0) (type default))
   )
+  (wire (pts (xy 111.76 66.04) (xy 111.76 68.58))
+    (stroke (width 0) (type default))
+  )
   (wire (pts (xy 10.16 97.79) (xy 10.16 20.32))
     (stroke (width 0) (type default))
   )
+  (wire (pts (xy 111.76 55.88) (xy 111.76 58.42))
+    (stroke (width 0) (type default))
+  )
+  (wire (pts (xy 111.76 50.8) (xy 111.76 53.34))
+    (stroke (width 0) (type default))
+  )
   (wire (pts (xy 10.16 105.41) (xy 10.16 100.33))
+    (stroke (width 0) (type default))
+  )
+  (wire (pts (xy 111.76 78.74) (xy 111.76 81.28))
+    (stroke (width 0) (type default))
+  )
+  (wire (pts (xy 111.76 68.58) (xy 111.76 71.12))
     (stroke (width 0) (type default))
   )
@@
         )
       )
+    )
+  )
+  (symbol (lib_id "power:GND") (at 111.76 86.36 0) (unit 1)
+    (in_bom yes) (on_board yes) (dnp no) (fields_autoplaced)
+    (property "Reference" "#PWR07" (at 111.76 92.71 0)
+      (effects (font (size 1.27 1.27)) hide)
+    )
+    (property "Value" "GND" (at 111.76 91.44 0)
+      (effects (font (size 1.27 1.27)))
+    )
+    (property "Footprint" "" (at 111.76 86.36 0)
+      (effects (font (size 1.27 1.27)) hide)
+    )
+    (property "Datasheet" "" (at 111.76 86.36 0)
+      (effects (font (size 1.27 1.27)) hide)
+    )
+    (pin "1")
+    (instances
+      (project "crush-pcb"
+        (path "/74b566fe-9d71-4817-95ed-d472d647f8c8"
+          (reference "#PWR07") (unit 1)
+        )
+      )
