File: i2c_level_shifter.kicad_sch (KiCad schematic)
At the start: 6 parts, among them Q1 BSN20, Q2 BSN20

Commit message: Deleted some unnecessary files that were renamed
Parts:
- R1, R2, R3, R4: footprint (none) -> Resistor_SMD:R_0402_1005Metric
Changed lines of the file:
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@@
       (effects (font (size 1.27 1.27)) (justify left))
     )
-    (property "Footprint" "" (at 39.116 15.494 90)
+    (property "Footprint" "Resistor_SMD:R_0402_1005Metric" (at 39.116 15.494 90)
       (effects (font (size 1.27 1.27)) hide)
     )
@@
     (pin "2")
     (instances
-      (project "crush-pcb"
+      (project "crush-main-board"
         (path "/74b566fe-9d71-4817-95ed-d472d647f8c8/063e1b7a-9baa-4271-8254-31d7d54fb281"
           (reference "R1") (unit 1)
@@
     (pin "3")
     (instances
-      (project "crush-pcb"
+      (project "crush-main-board"
         (path "/74b566fe-9d71-4817-95ed-d472d647f8c8/063e1b7a-9baa-4271-8254-31d7d54fb281"
           (reference "Q1") (unit 1)
@@
       (effects (font (size 1.27 1.27)) (justify left))
     )
-    (property "Footprint" "" (at 27.686 15.494 90)
+    (property "Footprint" "Resistor_SMD:R_0402_1005Metric" (at 27.686 15.494 90)
       (effects (font (size 1.27 1.27)) hide)
     )
@@
     (pin "2")
     (instances
-      (project "crush-pcb"
+      (project "crush-main-board"
         (path "/74b566fe-9d71-4817-95ed-d472d647f8c8/063e1b7a-9baa-4271-8254-31d7d54fb281"
           (reference "R2") (unit 1)
@@
       (effects (font (size 1.27 1.27)) (justify left))
     )
-    (property "Footprint" "" (at 74.676 15.494 90)
+    (property "Footprint" "Resistor_SMD:R_0402_1005Metric" (at 74.676 15.494 90)
       (effects (font (size 1.27 1.27)) hide)
     )
@@
     (pin "2")
     (instances
-      (project "crush-pcb"
+      (project "crush-main-board"
         (path "/74b566fe-9d71-4817-95ed-d472d647f8c8/063e1b7a-9baa-4271-8254-31d7d54fb281"
           (reference "R3") (unit 1)
@@
     (pin "3")
     (instances
-      (project "crush-pcb"
+      (project "crush-main-board"
         (path "/74b566fe-9d71-4817-95ed-d472d647f8c8/063e1b7a-9baa-4271-8254-31d7d54fb281"
           (reference "Q2") (unit 1)
@@
       (effects (font (size 1.27 1.27)) (justify left))
     )
-    (property "Footprint" "" (at 86.106 15.494 90)
+    (property "Footprint" "Resistor_SMD:R_0402_1005Metric" (at 86.106 15.494 90)
       (effects (font (size 1.27 1.27)) hide)
     )
@@
     (pin "2")
     (instances
-      (project "crush-pcb"
+      (project "crush-main-board"
         (path "/74b566fe-9d71-4817-95ed-d472d647f8c8/063e1b7a-9baa-4271-8254-31d7d54fb281"
           (reference "R4") (unit 1)

Commit message: Changed resistor and capacitor footprints to 0603
Parts:
- R1, R2, R3, R4: footprint Resistor_SMD:R_0402_1005Metric -> Resistor_SMD:R_0603_1608Metric_Pad0.98x0.95mm_HandSolder
Changed lines of the file:
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@@
       (effects (font (size 1.27 1.27)) (justify left))
     )
-    (property "Footprint" "Resistor_SMD:R_0402_1005Metric" (at 39.116 15.494 90)
+    (property "Footprint" "Resistor_SMD:R_0603_1608Metric_Pad0.98x0.95mm_HandSolder" (at 39.116 15.494 90)
       (effects (font (size 1.27 1.27)) hide)
     )
@@
       (effects (font (size 1.27 1.27)) (justify left))
     )
-    (property "Footprint" "Resistor_SMD:R_0402_1005Metric" (at 27.686 15.494 90)
+    (property "Footprint" "Resistor_SMD:R_0603_1608Metric_Pad0.98x0.95mm_HandSolder" (at 27.686 15.494 90)
       (effects (font (size 1.27 1.27)) hide)
     )
@@
       (effects (font (size 1.27 1.27)) (justify left))
     )
-    (property "Footprint" "Resistor_SMD:R_0402_1005Metric" (at 74.676 15.494 90)
+    (property "Footprint" "Resistor_SMD:R_0603_1608Metric_Pad0.98x0.95mm_HandSolder" (at 74.676 15.494 90)
       (effects (font (size 1.27 1.27)) hide)
     )
@@
       (effects (font (size 1.27 1.27)) (justify left))
     )
-    (property "Footprint" "Resistor_SMD:R_0402_1005Metric" (at 86.106 15.494 90)
+    (property "Footprint" "Resistor_SMD:R_0603_1608Metric_Pad0.98x0.95mm_HandSolder" (at 86.106 15.494 90)
       (effects (font (size 1.27 1.27)) hide)
     )

Commit message: update i2c level shifter
* Change resistors from 4.7k to 2.4k to improve signal quality
* Connect SCL MOSFET gate to 3.3V rather than 5V
Parts:
- R1, R2, R3, R4: value 4K7 -> 2k4
Connections:
- net 3V3: now also Q1.1 (G)
- net 5V: no longer Q1.1 (G)
Changed lines of the file:
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@@
   (junction (at 26.67 40.64) (diameter 0) (color 0 0 0 0)
   )
-  (junction (at 73.66 6.35) (diameter 0) (color 0 0 0 0)
-  )
   (junction (at 38.1 6.35) (diameter 0) (color 0 0 0 0)
   )
+  (junction (at 49.53 6.35) (diameter 0) (color 0 0 0 0)
+  )
   (junction (at 85.09 6.35) (diameter 0) (color 0 0 0 0)
   )
@@
     (stroke (width 0) (type default))
   )
-  (wire (pts (xy 73.66 6.35) (xy 62.23 6.35))
-    (stroke (width 0) (type default))
-  )
   (wire (pts (xy 73.66 26.67) (xy 100.965 26.67))
     (stroke (width 0) (type default))
@@
   )
   (wire (pts (xy 26.67 19.05) (xy 26.67 40.64))
+    (stroke (width 0) (type default))
+  )
+  (wire (pts (xy 49.53 6.35) (xy 62.23 6.35))
     (stroke (width 0) (type default))
   )
@@
   (symbol (lib_id "Device:R_US") (at 38.1 15.24 0) (unit 1)
     (in_bom yes) (on_board yes) (dnp no) (fields_autoplaced)
-    (property "Reference" "R1" (at 40.64 14.605 0)
-      (effects (font (size 1.27 1.27)) (justify left))
-    )
-    (property "Value" "4K7" (at 40.64 17.145 0)
+    (property "Reference" "R1" (at 40.64 13.97 0)
+      (effects (font (size 1.27 1.27)) (justify left))
+    )
+    (property "Value" "2k4" (at 40.64 16.51 0)
       (effects (font (size 1.27 1.27)) (justify left))
     )
@@
   (symbol (lib_id "Device:R_US") (at 26.67 15.24 0) (unit 1)
     (in_bom yes) (on_board yes) (dnp no) (fields_autoplaced)
-    (property "Reference" "R2" (at 29.21 14.605 0)
-      (effects (font (size 1.27 1.27)) (justify left))
-    )
-    (property "Value" "4K7" (at 29.21 17.145 0)
+    (property "Reference" "R2" (at 29.21 13.97 0)
+      (effects (font (size 1.27 1.27)) (justify left))
+    )
+    (property "Value" "2k4" (at 29.21 16.51 0)
       (effects (font (size 1.27 1.27)) (justify left))
     )
@@
   (symbol (lib_id "Device:R_US") (at 73.66 15.24 0) (unit 1)
     (in_bom yes) (on_board yes) (dnp no) (fields_autoplaced)
-    (property "Reference" "R3" (at 76.2 14.605 0)
-      (effects (font (size 1.27 1.27)) (justify left))
-    )
-    (property "Value" "4K7" (at 76.2 17.145 0)
+    (property "Reference" "R3" (at 76.2 13.97 0)
+      (effects (font (size 1.27 1.27)) (justify left))
+    )
+    (property "Value" "2k4" (at 76.2 16.51 0)
       (effects (font (size 1.27 1.27)) (justify left))
     )
@@
   (symbol (lib_id "Device:R_US") (at 85.09 15.24 0) (unit 1)
     (in_bom yes) (on_board yes) (dnp no) (fields_autoplaced)
-    (property "Reference" "R4" (at 87.63 14.605 0)
-      (effects (font (size 1.27 1.27)) (justify left))
-    )
-    (property "Value" "4K7" (at 87.63 17.145 0)
-      (effects (font (size 1.27 1.27)) (justify left))
-    )
+    (property "Reference" "R4" (at 87.63 13.97 0)
+      (effects (font (size 1.27 1.27)) (justify left))
+    )
+    (property "Value" "2k4" (at 87.63 16.51 0)
+      (effects (font (size 1.27 1.27)) (justify left))
+    )
