File: crush-main-board.kicad_sch (KiCad schematic)
At the start: 38 parts, among them J1 4x4_Header, J10 3x3 Header, J11 3x3 Header, J12 3x2 Header, J13 3x4_Header, J14 3x4_Header, J15 2157601008, J16 Conn_01x02, J17 Conn_01x02, J18 Conn_Coaxial, J2 4x4_Header, J3 6x2_Header, J4 3x1_Header, J5 3x2 Header, J6 3x2 Header, J7 3x4 Header, J8 3x4 Header, J9 3x3 Header, SW1 SW_SPST, U1 Teensy4.1, U2 ISO7740DW, U3 ISO7740DW, U4 ISO1640BDR, U5 INA232B, U6 INA232B

Commit message: Remove uninteresting test points (all)
Other:
- note added: "swap this with 3v3?"
- moved on the sheet: SW1
Changed lines of the file:
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@@
 		)
 	)
+	(text "swap this with 3v3?"
+		(exclude_from_sim no)
+		(at 255.778 77.47 0)
+		(effects
+			(font
+				(size 1.27 1.27)
+			)
+		)
+	)
 	(text "I2C Addr: 0x48"
 		(exclude_from_sim no)
@@
 	(text_box "On-board Kill Switch\n"
 		(exclude_from_sim no)
-		(at 226.695 180.34 0)
+		(at 333.375 106.68 0)
 		(size 38.1 24.13)
 		(margins 1.5 1.5 1.5 1.5)
@@
 		(at 78.74 83.82)
 	)
+	(bus_entry
+		(at 162.56 260.35)
+		(size 2.54 2.54)
+		(stroke
+			(width 0)
+			(type default)
+		)
+	)
+	(bus_entry
+		(at 59.69 303.53)
+		(size 2.54 2.54)
+		(stroke
+			(width 0)
+			(type default)
+		)
+	)
 	(wire
 		(pts
@@
 	(wire
 		(pts
-			(xy 234.95 199.39) (xy 245.11 199.39)
+			(xy 341.63 125.73) (xy 351.79 125.73)
 		)
 		(stroke
@@
 	(wire
 		(pts
-			(xy 234.95 186.69) (xy 234.95 187.96)
+			(xy 341.63 113.03) (xy 341.63 114.3)
 		)
 		(stroke
@@
 	(wire
 		(pts
-			(xy 234.95 199.39) (xy 234.95 198.12)
+			(xy 341.63 125.73) (xy 341.63 124.46)
 		)
 		(stroke
@@
 	(wire
 		(pts
-			(xy 234.95 186.69) (xy 245.11 186.69)
+			(xy 341.63 113.03) (xy 351.79 113.03)
 		)
 		(stroke
@@
 	(global_label "HW_KILL_3"
 		(shape input)
-		(at 245.11 186.69 0)
+		(at 351.79 113.03 0)
 		(fields_autoplaced yes)
 		(effects
@@
 		)
 		(property "Intersheetrefs" "${INTERSHEET_REFS}"
-			(at 257.9528 186.69 0)
+			(at 364.6328 113.03 0)
 			(hide yes)
 			(show_name no)
@@
 	(global_label "HW_KILL_4"
 		(shape input)
-		(at 245.11 199.39 0)
+		(at 351.79 125.73 0)
 		(fields_autoplaced yes)
 		(effects
@@
 		)
 		(property "Intersheetrefs" "${INTERSHEET_REFS}"
-			(at 257.9528 199.39 0)
+			(at 364.6328 125.73 0)
 			(hide yes)
 			(show_name no)
@@
 	(symbol
 		(lib_id "Switch:SW_SPST")
-		(at 234.95 193.04 90)
+		(at 341.63 119.38 90)
 		(unit 1)
 		(body_style 1)
@@
 		(fields_autoplaced yes)
 		(property "Reference" "SW1"
-			(at 236.22 191.7699 90)
+			(at 342.9 118.1099 90)
 			(show_name no)
 			(do_not_autoplace no)
@@
 		)
 		(property "Value" "SW_SPST"
-			(at 236.22 194.3099 90)
+			(at 342.9 120.6499 90)
 			(show_name no)
 			(do_not_autoplace no)
@@
 		)
 		(property "Footprint" "Button_Switch_SMD:SW_DIP_SPSTx01_Slide_9.78x4.72mm_W8.61mm_P2.54mm"
-			(at 234.95 193.04 0)
+			(at 341.63 119.38 0)
 			(hide yes)
 			(show_name no)
@@
 		)
 		(property "Datasheet" ""
-			(at 234.95 193.04 0)
+			(at 341.63 119.38 0)
 			(hide yes)
 			(show_name no)
@@
 		)
 		(property "Description" "Single Pole Single Throw (SPST) switch"
-			(at 234.95 193.04 0)
+			(at 341.63 119.38 0)
 			(hide yes)
 			(show_name no)
